Commit message: fix falling angle for reward calculation

File: data/urdf/robots/mooncake/urdf/mooncake.xacro (robot description, xacro)
@@ -3,5 +3,5 @@
 	xmlns:xacro="http://ros.org/wiki/xacro">
 	<!--Rotate entire robot-->
-    <xacro:property name="robot_angle" value="${-pi/2}"/>
+    <xacro:property name="robot_angle" value="${0}"/>
 	<xacro:macro name="inertial_box" params="size rho:=1000 xyz:='0 0 0' rpy:='0 0 0'">
 		<xacro:property name="w" value="${size.split()[0]}"/>
