Commit message: change mooncake's part material name
ถ้าชื่อ material ที่สร้างมาจาก blender ซำ้กันจะทำให้ isaac sim งงตอน import URDF

File: data/urdf/robots/mooncake/urdf/mooncake.urdf (robot description, URDF)
Before this commit: robot mooncake, 77 links, 76 joints
Links:
- link base_plate: geometry collision cylinder length=0.006 radius=0.15; visual mesh filename=package://meshes/lower_plate.dae scale=1 1 1
- link motor_0: geometry collision cylinder length=0.11 radius=0.019; visual mesh filename=package://meshes/ZGX38REE.dae scale=1 1 1
- link motor_1: geometry collision cylinder length=0.11 radius=0.019; visual mesh filename=package://meshes/ZGX38REE.dae scale=1 1 1
- link motor_2: geometry collision cylinder length=0.11 radius=0.019; visual mesh filename=package://meshes/ZGX38REE.dae scale=1 1 1
- link motor_mount_0: geometry visual mesh filename=package://meshes/motor_mount.dae scale=1 1 1
- link motor_mount_1: geometry visual mesh filename=package://meshes/motor_mount.dae scale=1 1 1
- link motor_mount_2: geometry visual mesh filename=package://meshes/motor_mount.dae scale=1 1 1
- link pillar_0: geometry collision box size=0.0225 0.006 0.174; visual mesh filename=package://meshes/pillar.dae scale=1 1 1
- link pillar_1: geometry collision box size=0.0225 0.006 0.174; visual mesh filename=package://meshes/pillar.dae scale=1 1 1
- link pillar_10: geometry collision box size=0.0225 0.006 0.174; visual mesh filename=package://meshes/pillar.dae scale=1 1 1
- link pillar_11: geometry collision box size=0.0225 0.006 0.174; visual mesh filename=package://meshes/pillar.dae scale=1 1 1
- link pillar_2: geometry collision box size=0.0225 0.006 0.174; visual mesh filename=package://meshes/pillar.dae scale=1 1 1
- link pillar_3: geometry collision box size=0.0225 0.006 0.174; visual mesh filename=package://meshes/pillar.dae scale=1 1 1
- link pillar_4: geometry collision box size=0.0225 0.006 0.174; visual mesh filename=package://meshes/pillar.dae scale=1 1 1
- link pillar_5: geometry collision box size=0.0225 0.006 0.174; visual mesh filename=package://meshes/pillar.dae scale=1 1 1
- link pillar_6: geometry collision box size=0.0225 0.006 0.174; visual mesh filename=package://meshes/pillar.dae scale=1 1 1
- link pillar_7: geometry collision box size=0.0225 0.006 0.174; visual mesh filename=package://meshes/pillar.dae scale=1 1 1
- link pillar_8: geometry collision box size=0.0225 0.006 0.174; visual mesh filename=package://meshes/pillar.dae scale=1 1 1
- link pillar_9: geometry collision box size=0.0225 0.006 0.174; visual mesh filename=package://meshes/pillar.dae scale=1 1 1
- link upper_plate: geometry collision cylinder length=0.006 radius=0.15; visual mesh filename=package://meshes/upper_plate.dae scale=1 1 1
- link wheel_0: geometry visual mesh filename=package://meshes/omni_wheel.dae scale=1 1 1
- link wheel_1: geometry visual mesh filename=package://meshes/omni_wheel.dae scale=1 1 1
- link wheel_2: geometry visual mesh filename=package://meshes/omni_wheel.dae scale=1 1 1

File: data/urdf/robots/mooncake/urdf/mooncake.xacro (robot description, xacro)
@@ -65,5 +65,5 @@
 			<visual>
 				<geometry>
-					<mesh filename="/media/teera/ROGESD/urdf/robots/mooncake/meshes/pillar.dae" scale="1 1 1"/>
+					<mesh filename="package://meshes/pillar.dae" scale="1 1 1"/>
 				</geometry>
 			</visual>
@@ -125,5 +125,5 @@
 			<visual>
 				<geometry>
-					<mesh filename="/media/teera/ROGESD/urdf/robots/mooncake/meshes/omni_wheel.dae" scale="1 1 1"/>
+					<mesh filename="package://meshes/omni_wheel.dae" scale="1 1 1"/>
 				</geometry>
 			</visual>
@@ -165,5 +165,5 @@
 			<visual>
 				<geometry>
-					<mesh filename="/media/teera/ROGESD/urdf/robots/mooncake/meshes/ZGX38REE.dae" scale="1 1 1"/>
+					<mesh filename="package://meshes/ZGX38REE.dae" scale="1 1 1"/>
 				</geometry>
 			</visual>
@@ -186,5 +186,5 @@
 			<visual>
 				<geometry>
-					<mesh filename="/media/teera/ROGESD/urdf/robots/mooncake/meshes/motor_mount.dae" scale="1 1 1"/>
+					<mesh filename="package://meshes/motor_mount.dae" scale="1 1 1"/>
 				</geometry>
 			</visual>
@@ -202,5 +202,5 @@
 		<visual>
 			<geometry>
-				<mesh filename="/media/teera/ROGESD/urdf/robots/mooncake/meshes/lower_plate.dae" scale="1 1 1"/>
+				<mesh filename="package://meshes/lower_plate.dae" scale="1 1 1"/>
 			</geometry>
 		</visual>
@@ -213,5 +213,5 @@
 		<visual>
 			<geometry>
-				<mesh filename="/media/teera/ROGESD/urdf/robots/mooncake/meshes/upper_plate.dae" scale="1 1 1"/>
+				<mesh filename="package://meshes/upper_plate.dae" scale="1 1 1"/>
 			</geometry>
 		</visual>

Commit message: correct motor_angle in mooncake.xacro

File: data/urdf/robots/mooncake/urdf/mooncake.urdf (robot description, URDF)
Before this commit: robot mooncake, 77 links, 76 joints
Joints:
- joint motor_0_joint: origin xyz=-0.029504429610734115 0 0.006062754129380309 rpy=0 -0.8726646259971648 0 -> xyz=-0.033202134613707274 0 -0.003797792545214791 rpy=0 -0.6981317007977318 0
- joint motor_1_joint: origin xyz=-0.029504429610734115 0 0.006062754129380309 rpy=0 -0.8726646259971648 0 -> xyz=-0.033202134613707274 0 -0.003797792545214791 rpy=0 -0.6981317007977318 0
- joint motor_2_joint: origin xyz=-0.029504429610734115 0 0.006062754129380309 rpy=0 -0.8726646259971648 0 -> xyz=-0.033202134613707274 0 -0.003797792545214791 rpy=0 -0.6981317007977318 0

File: data/urdf/robots/mooncake/urdf/mooncake.xacro (robot description, xacro)
@@ -157,5 +157,5 @@
 	<xacro:macro name="motor_assembly" params="num angle">
 		<!--Angle between base and motor (50 degree from floor)-->
-		<xacro:property name="motor_angle" value="${5*pi/18}"/>
+		<xacro:property name="motor_angle" value="${4*pi/18}"/>
 		<!--Extended radius from center (referenced to each motor mount)-->
 		<xacro:property name="delta_r" value="${0.025-0.025*sin(motor_angle)-0.055*cos(motor_angle)}"/>

Commit message: move wheel position & simplify RL action
move wheel position
- 0: upper
- 1: lower left
- 2: lower right
simplify RL action
- use robot's wheel kinematics to simplify RL action from 3 -> 2
- omega_0 = (v_x-d*w_z)/r
- omega_1 = -(v_x-math.sqrt(3)*v_y+2*d*w_z)/(2*r)
- omega_2 = -(v_x+math.sqrt(3)*v_y+2*d*w_z)/(2*r)

File: data/urdf/robots/mooncake/urdf/mooncake.urdf (robot description, URDF)
Before this commit: robot mooncake, 77 links, 76 joints
Joints:
- joint motor_mount_0_joint: origin xyz=-0.095 -1.1634144591899856e-17 0 rpy=0 0 -3.141592653589793 -> xyz=-1.745121688784978e-17 0.095 0 rpy=0 0 -4.71238898038469
- joint motor_mount_1_joint: origin xyz=0.047500000000000014 -0.08227241335952167 0 rpy=0 0 -1.0471975511965976 -> xyz=-0.08227241335952165 -0.047500000000000035 0 rpy=0 0 -2.617993877991494
- joint motor_mount_2_joint: origin xyz=0.047500000000000014 0.08227241335952167 0 rpy=0 0 1.0471975511965976 -> xyz=0.08227241335952167 -0.0475 0 rpy=0 0 -0.5235987755982989
- joint pillar_0_joint: origin xyz=0.13125 0.022 0.08425 rpy=0 0 0.0 -> xyz=0.022000000000000006 -0.13125 0.08425 rpy=0 0 -1.5707963267948966
- joint pillar_10_joint: origin xyz=0.08467755888325758 -0.10266583424670765 0.08425 rpy=0 0 5.235987755982988 -> xyz=-0.10266583424670765 -0.08467755888325758 0.08425 rpy=0 0 3.6651914291880914
- joint pillar_11_joint: origin xyz=0.04657244111674226 -0.12466583424670762 0.08425 rpy=0 0 5.235987755982988 -> xyz=-0.12466583424670762 -0.04657244111674226 0.08425 rpy=0 0 3.6651914291880914
- joint pillar_1_joint: origin xyz=0.13125 -0.022 0.08425 rpy=0 0 0.0 -> xyz=-0.021999999999999992 -0.13125 0.08425 rpy=0 0 -1.5707963267948966
- joint pillar_2_joint: origin xyz=0.04657244111674237 0.12466583424670757 0.08425 rpy=0 0 1.0471975511965976 -> xyz=0.12466583424670756 -0.04657244111674236 0.08425 rpy=0 0 -0.5235987755982989
- joint pillar_3_joint: origin xyz=0.08467755888325766 0.10266583424670757 0.08425 rpy=0 0 1.0471975511965976 -> xyz=0.10266583424670755 -0.08467755888325765 0.08425 rpy=0 0 -0.5235987755982989
- joint pillar_4_joint: origin xyz=-0.08467755888325762 0.10266583424670758 0.08425 rpy=0 0 2.0943951023931953 -> xyz=0.10266583424670758 0.08467755888325762 0.08425 rpy=0 0 0.5235987755982987
- joint pillar_5_joint: origin xyz=-0.04657244111674232 0.12466583424670757 0.08425 rpy=0 0 2.0943951023931953 -> xyz=0.12466583424670757 0.04657244111674232 0.08425 rpy=0 0 0.5235987755982987
- joint pillar_6_joint: origin xyz=-0.13125 -0.02199999999999998 0.08425 rpy=0 0 3.141592653589793 -> xyz=-0.021999999999999992 0.13125 0.08425 rpy=0 0 1.5707963267948966
- joint pillar_7_joint: origin xyz=-0.13125 0.022000000000000016 0.08425 rpy=0 0 3.141592653589793 -> xyz=0.022000000000000006 0.13125 0.08425 rpy=0 0 1.5707963267948966
- joint pillar_8_joint: origin xyz=-0.046572441116742413 -0.12466583424670755 0.08425 rpy=0 0 4.1887902047863905 -> xyz=-0.12466583424670756 0.0465724411167424 0.08425 rpy=0 0 2.617993877991494
- joint pillar_9_joint: origin xyz=-0.0846775588832577 -0.10266583424670753 0.08425 rpy=0 0 4.1887902047863905 -> xyz=-0.10266583424670754 0.08467755888325769 0.08425 rpy=0 0 2.617993877991494
- joint upper_plate_joint: origin xyz=0 0 0.1685 -> xyz=0 0 0.1685 rpy=0 0 -1.5707963267948966
- joint wheel_0_joint: axis 0 0 1 -> 0 0 -1
- joint wheel_1_joint: axis 0 0 1 -> 0 0 -1
- joint wheel_2_joint: axis 0 0 1 -> 0 0 -1

File: data/urdf/robots/mooncake/urdf/mooncake.xacro (robot description, xacro)
@@ -2,5 +2,7 @@
 <robot name="mooncake"
 	xmlns:xacro="http://ros.org/wiki/xacro">
-    <xacro:macro name="inertial_box" params="size rho:=1000 xyz:='0 0 0' rpy:='0 0 0'">
+	<!--Rotate entire robot-->
+    <xacro:property name="robot_angle" value="${-pi/2}"/>
+	<xacro:macro name="inertial_box" params="size rho:=1000 xyz:='0 0 0' rpy:='0 0 0'">
 		<xacro:property name="w" value="${size.split()[0]}"/>
 		<xacro:property name="d" value="${size.split()[1]}"/>
@@ -79,5 +81,5 @@
     <xacro:macro name="pillars" params="num">
 		<!--Angle from center-->
-		<xacro:property name="angle" value="${num*(pi/3)}"/>
+		<xacro:property name="angle" value="${num*(pi/3) + robot_angle}"/>
 		<!--Radius from center-->
 		<xacro:property name="r" value="0.13125"/>
@@ -132,5 +134,5 @@
 		<joint name="wheel_${num}_joint" type="continuous">
 			<origin xyz="0 0 ${z}" rpy="0 0 0"/>
-			<axis xyz="0 0 1"/>
+			<axis xyz="0 0 -1"/>
 			<parent link="motor_${num}"/>
 			<child link="wheel_${num}"/>
@@ -180,5 +182,5 @@
 	<xacro:macro name="motor_mount_assembly" params="num">
 		<!--Angle from center-->
-		<xacro:property name="angle" value="${(num-1.5)*(2*pi/3)}"/>
+		<xacro:property name="angle" value="${(num-3/2)*(2*pi/3) + robot_angle}"/>
 		<!--Radius from center-->
 		<xacro:property name="r" value="0.095"/>
@@ -201,4 +203,5 @@
 	<link name="base_plate">
 		<visual>
+			<origin rpy="0 0 ${robot_angle}"/>
 			<geometry>
 				<mesh filename="package://meshes/lower_plate.dae" scale="1 1 1"/>
@@ -220,5 +223,5 @@
 	</link>
 	<joint name="upper_plate_joint" type="fixed">
-		<origin xyz="0 0 0.1685"/>
+		<origin xyz="0 0 0.1685" rpy="0 0 ${robot_angle}"/>
 		<parent link="base_plate"/>
 		<child link="upper_plate"/>

Commit message: update mooncake can be stable in a short time

File: data/urdf/robots/mooncake/urdf/mooncake.urdf (robot description, URDF)
Before this commit: robot mooncake, 77 links, 76 joints
Joints:
- joint motor_mount_0_joint: origin xyz=-1.745121688784978e-17 0.095 0 rpy=0 0 -4.71238898038469 -> xyz=-0.095 -1.1634144591899856e-17 0 rpy=0 0 -3.141592653589793
- joint motor_mount_1_joint: origin xyz=-0.08227241335952165 -0.047500000000000035 0 rpy=0 0 -2.617993877991494 -> xyz=0.047500000000000014 -0.08227241335952167 0 rpy=0 0 -1.0471975511965976
- joint motor_mount_2_joint: origin xyz=0.08227241335952167 -0.0475 0 rpy=0 0 -0.5235987755982989 -> xyz=0.047500000000000014 0.08227241335952167 0 rpy=0 0 1.0471975511965976
- joint pillar_0_joint: origin xyz=0.022000000000000006 -0.13125 0.08425 rpy=0 0 -1.5707963267948966 -> xyz=0.13125 0.022 0.08425 rpy=0 0 0.0
- joint pillar_10_joint: origin xyz=-0.10266583424670765 -0.08467755888325758 0.08425 rpy=0 0 3.6651914291880914 -> xyz=0.08467755888325758 -0.10266583424670765 0.08425 rpy=0 0 5.235987755982988
- joint pillar_11_joint: origin xyz=-0.12466583424670762 -0.04657244111674226 0.08425 rpy=0 0 3.6651914291880914 -> xyz=0.04657244111674226 -0.12466583424670762 0.08425 rpy=0 0 5.235987755982988
- joint pillar_1_joint: origin xyz=-0.021999999999999992 -0.13125 0.08425 rpy=0 0 -1.5707963267948966 -> xyz=0.13125 -0.022 0.08425 rpy=0 0 0.0
- joint pillar_2_joint: origin xyz=0.12466583424670756 -0.04657244111674236 0.08425 rpy=0 0 -0.5235987755982989 -> xyz=0.04657244111674237 0.12466583424670757 0.08425 rpy=0 0 1.0471975511965976
- joint pillar_3_joint: origin xyz=0.10266583424670755 -0.08467755888325765 0.08425 rpy=0 0 -0.5235987755982989 -> xyz=0.08467755888325766 0.10266583424670757 0.08425 rpy=0 0 1.0471975511965976
- joint pillar_4_joint: origin xyz=0.10266583424670758 0.08467755888325762 0.08425 rpy=0 0 0.5235987755982987 -> xyz=-0.08467755888325762 0.10266583424670758 0.08425 rpy=0 0 2.0943951023931953
- joint pillar_5_joint: origin xyz=0.12466583424670757 0.04657244111674232 0.08425 rpy=0 0 0.5235987755982987 -> xyz=-0.04657244111674232 0.12466583424670757 0.08425 rpy=0 0 2.0943951023931953
- joint pillar_6_joint: origin xyz=-0.021999999999999992 0.13125 0.08425 rpy=0 0 1.5707963267948966 -> xyz=-0.13125 -0.02199999999999998 0.08425 rpy=0 0 3.141592653589793
- joint pillar_7_joint: origin xyz=0.022000000000000006 0.13125 0.08425 rpy=0 0 1.5707963267948966 -> xyz=-0.13125 0.022000000000000016 0.08425 rpy=0 0 3.141592653589793
- joint pillar_8_joint: origin xyz=-0.12466583424670756 0.0465724411167424 0.08425 rpy=0 0 2.617993877991494 -> xyz=-0.046572441116742413 -0.12466583424670755 0.08425 rpy=0 0 4.1887902047863905
- joint pillar_9_joint: origin xyz=-0.10266583424670754 0.08467755888325769 0.08425 rpy=0 0 2.617993877991494 -> xyz=-0.0846775588832577 -0.10266583424670753 0.08425 rpy=0 0 4.1887902047863905
- joint upper_plate_joint: origin xyz=0 0 0.1685 rpy=0 0 -1.5707963267948966 -> xyz=0 0 0.1685
- joint wheel_0_joint: axis 0 0 -1 -> 0 0 1
- joint wheel_1_joint: axis 0 0 -1 -> 0 0 1
- joint wheel_2_joint: axis 0 0 -1 -> 0 0 1

Commit message: fix import mooncake (instanceable)

File: data/urdf/robots/mooncake/urdf/mooncake.urdf (robot description, URDF)
Before this commit: robot mooncake, 77 links, 76 joints
Joints:
- joint upper_plate_joint: origin xyz=0 0 0.1685 -> xyz=0 0 0.1685 rpy=0 0 0
- joint wheel_0_joint: axis 0 0 1 -> 0 0 -1
- joint wheel_1_joint: axis 0 0 1 -> 0 0 -1
- joint wheel_2_joint: axis 0 0 1 -> 0 0 -1
