Commit message: finalized visual in obike.xacro & meshes

File: data/urdf/robots/obike/urdf/obike.urdf (robot description, URDF)
Before this commit: robot obike, 6 links, 5 joints
Links:
- removed link base
- removed link body
- removed link reaction_wheel_assembly
- removed link wheel_0
- removed link wheel_1
- added link chassic; visual mesh filename=/home/fiborobotlab/urdf/robots/obike/meshes/chassic.dae scale=1 1 1
- added link faulhaber; visual mesh filename=/home/fiborobotlab/urdf/robots/obike/meshes/faulhaber.dae scale=1 1 1
- added link front_chassic; visual mesh filename=/home/fiborobotlab/urdf/robots/obike/meshes/front_chassic.d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 scale=1 1 1
- added link front_wheel; visual mesh filename=/home/fiborobotlab/urdf/robots/obike/meshes/front_wheel.dae scale=1 1 1
- added link front_wheel_arm; visual mesh filename=/home/fiborobotlab/urdf/robots/obike/meshes/front_wheel_arm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 scale=1 1 1
- added link motor_mount; visual mesh filename=/home/fiborobotlab/urdf/robots/obike/meshes/motor_mount.dae scale=1 1 1
- added link reaction_wheel_steel; visual mesh filename=/home/fiborobotlab/urdf/robots/obike/meshes/reaction_wheel_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 scale=1 1 1
- added link rear_wheel; visual mesh filename=/home/fiborobotlab/urdf/robots/obike/meshes/rear_wheel.dae scale=1 1 1
- link reaction_wheel: mass 0.19800011006761326 -> None; geometry visual mesh filename=/home/fiborobotlab/urdf/robots/obike/meshes/reaction_wheel.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 scale=1 1 1
Joints:
- removed joint base_joint
- removed joint reaction_wheel_assembly_joint
- removed joint wheel_0_joint
- removed joint wheel_1_joint
- added joint faulhaber_joint: type fixed, parent motor_mount, child faulhaber, origin xyz=0 0 0 rpy=0 1.5707963267948966 0
- added joint front_chassic_joint: type fixed, parent chassic, child front_chassic, origin xyz=0.055 0 0.035 rpy=0 0 0
- added joint front_wheel_arm_joint: type continuous, parent chassic, child front_wheel_arm, origin xyz=0.107304 0 0.03901 rpy=0 2.6179938779914944 0, axis 0 0 1
- added joint front_wheel_joint: type continuous, parent front_wheel_arm, child front_wheel, origin xyz=0 0 0.035 rpy=-1.5707963267948966 0 0, axis 0 0 1
- added joint motor_mount_joint: type fixed, parent chassic, child motor_mount, origin xyz=-0.005 0 0.08 rpy=0 0 0
- added joint reaction_wheel_steel_joint: type fixed, parent reaction_wheel, child reaction_wheel_steel, origin xyz=0 0 0.004 rpy=0 0 0
- added joint rear_wheel_joint: type continuous, parent chassic, child rear_wheel, origin xyz=-0.05 0 0.022 rpy=1.5707963267948966 0 0, axis 0 0 1
- joint reaction_wheel_joint: origin xyz=0 0 0.05 rpy=0 0 0 -> xyz=0.044 0 0 rpy=0 1.5707963267948966 0; parent reaction_wheel_assembly -> motor_mount

File: data/urdf/robots/obike/urdf/obike.xacro (robot description, xacro)
@@ -1,4 +1,5 @@
 <?xml version="1.0"?>
 <robot name="obike" xmlns:xacro="http://ros.org/wiki/xacro">
+	<xacro:property name="MODEL_PATH" value="/home/fiborobotlab/urdf/robots/obike/meshes/"/>
     <xacro:macro name="inertial_box" params="size rho:=1000 xyz:='0 0 0' rpy:='0 0 0'">
 		<xacro:property name="w" value="${size.split()[0]}"/>
@@ -60,71 +61,117 @@
 		</collision>
 	</xacro:macro>
-	<link name="base">
-	</link>
-    <link name="body">
+	<xacro:macro name="inertial_manual" params="mass xyz:='0 0 0' rpy:='0 0 0' ixx iyy izz ixy:='0' ixz:='0' iyz:='0'">
+		<inertial>
+			<origin xyz="${xyz}" rpy="${rpy}"/>
+			<mass value="${mass}"/>
+			<inertia ixx="${ixx}" iyy="${iyy}" izz="${izz}" ixy="${ixy}" ixz="${ixz}" iyz="${iyz}"/>
+		</inertial>
+	</xacro:macro>
+	<link name="chassic">
 		<visual>
-			<origin xyz="0 0 0" rpy="0 0 0"/>
 			<geometry>
-				<box size="0.150 0.04 0.06" xyz="0 0 0"/>
+				<mesh filename="${MODEL_PATH}chassic.dae" scale="1 1 1"/>
 			</geometry>
 		</visual>
-		<!-- <xacro:collision_box size="0.150 0.04 0.06"/> -->
-		<xacro:inertial_box size="0.150 0.04 0.06" rho="513.89"/>
 	</link>
-    <joint name="base_joint" type="continuous">
-        <origin xyz="0 0 0.0665" rpy="0 0 0"/>
-        <axis xyz="1 0 0"/>
-		<parent link="base"/>
-		<child link="body"/>
-    </joint>
-	<link name="reaction_wheel_assembly">
+	<link name="motor_mount">
 		<visual>
-			<origin rpy="0 0 0"/>
 			<geometry>
-				<cylinder xyz="0 0 0" rpy="0 0 0" radius="0.0125" length="0.08"/>
+				<mesh filename="${MODEL_PATH}motor_mount.dae" scale="1 1 1"/>
 			</geometry>
 		</visual>
-		<!-- motor inertia -->
-		<xacro:inertial_cylinder rho="5424" length="0.08" radius="0.0125"/>
 	</link>
-    <joint name="reaction_wheel_assembly_joint" type="fixed">
-        <origin xyz="0 0 0.0605" rpy="0 ${pi/2} 0"/>
-        <parent link="body"/>
-		<child link="reaction_wheel_assembly"/>
-    </joint>
+	<joint name="motor_mount_joint" type="fixed">
+		<origin xyz="-0.005 0 0.08" rpy="0 0 0"/>
+		<parent link="chassic"/>
+		<child link="motor_mount"/>
+	</joint>
+	<link name="front_chassic">
+		<visual>
+			<geometry>
+				<mesh filename="${MODEL_PATH}front_chassic.dae" scale="1 1 1"/>
+			</geometry>
+		</visual>
+	</link>
+	<joint name="front_chassic_joint" type="fixed">
+		<origin xyz="0.055 0 0.035" rpy="0 0 0"/>
+		<parent link="chassic"/>
+		<child link="front_chassic"/>
+	</joint>
+	<link name="front_wheel_arm">
+		<visual>
+			<geometry>
+				<mesh filename="${MODEL_PATH}front_wheel_arm.dae" scale="1 1 1"/>
+			</geometry>
+		</visual>
+	</link>
+	<joint name="front_wheel_arm_joint" type="continuous">
+		<origin xyz="0.107304 0 0.03901" rpy="0 ${5*pi/6} 0"/>
+		<axis xyz="0 0 1"/>
+		<parent link="chassic"/>
+		<child link="front_wheel_arm"/>
+	</joint>
+	<link name="front_wheel">
+		<visual>
+			<geometry>
+				<mesh filename="${MODEL_PATH}front_wheel.dae" scale="1 1 1"/>
+			</geometry>
+		</visual>
+	</link>
+	<joint name="front_wheel_joint" type="continuous">
+		<origin xyz="0 0 0.035" rpy="${-pi/2} 0 0"/>
+		<axis xyz="0 0 1"/>
+		<parent link="front_wheel_arm"/>
+		<child link="front_wheel"/>
+	</joint>
+	<link name="faulhaber">
+		<visual>
+			<geometry>
+				<mesh filename="${MODEL_PATH}faulhaber.dae" scale="1 1 1"/>
+			</geometry>
+		</visual>
+	</link>
+	<joint name="faulhaber_joint" type="fixed">
+		<origin xyz="0 0 0" rpy="0 ${pi/2} 0"/>
+		<parent link="motor_mount"/>
+		<child link="faulhaber"/>
+	</joint>
 	<link name="reaction_wheel">
 		<visual>
-			<origin rpy="0 0 0"/>
 			<geometry>
-				<cylinder xyz="0 0 0" rpy="0 0 0" radius="0.035" length="0.01"/>
+				<mesh filename="${MODEL_PATH}reaction_wheel.dae" scale="1 1 1"/>
 			</geometry>
 		</visual>
-		<!-- reaction wheel inertia -->
-		<xacro:inertial_cylinder rho="5144.93" length="0.01" radius="0.035"/>
 	</link>
 	<joint name="reaction_wheel_joint" type="continuous">
-		<origin xyz="0 0 0.05" rpy="0 0 0"/>
-        <axis xyz="0 0 1"/>
-		<parent link="reaction_wheel_assembly"/>
+		<origin xyz="0.044 0 0" rpy="0 ${pi/2} 0"/>
+		<axis xyz="0 0 1"/>
+		<parent link="motor_mount"/>
 		<child link="reaction_wheel"/>
 	</joint>
-	<xacro:macro name="wheel" params="num xyz">
-		<link name="wheel_${num}">
-			<visual>
-				<geometry>
-					<cylinder xyz="0 0 0" rpy="0 0 0" radius="0.0365" length="0.001"/>
-				</geometry>
-			</visual>
-			<xacro:collision_cylinder radius="0.0365" length="0.001"/>
-			<xacro:inertial_cylinder rho="1000" radius="0.0365" length="0.001"/>
-		</link>
-		<joint name="wheel_${num}_joint" type="continuous">
-			<origin xyz="${xyz}" rpy="${pi/2} 0 0"/>
-			<axis xyz="0 0 1"/>
-			<parent link="body"/>
-			<child link="wheel_${num}"/>
-		</joint>
-	</xacro:macro>
-	<xacro:wheel num="0" xyz="-0.05 0 -0.0365"/>
-	<xacro:wheel num="1" xyz="0.05 0 -0.0365"/>
+	<link name="reaction_wheel_steel">
+		<visual>
+			<geometry>
+				<mesh filename="${MODEL_PATH}reaction_wheel_steel.dae" scale="1 1 1"/>
+			</geometry>
+		</visual>
+	</link>
+	<joint name="reaction_wheel_steel_joint" type="fixed">
+		<origin xyz="0 0 0.004" rpy="0 0 0"/>
+		<parent link="reaction_wheel"/>
+		<child link="reaction_wheel_steel"/>
+	</joint>
+	<link name="rear_wheel">
+		<visual>
+			<geometry>
+				<mesh filename="${MODEL_PATH}rear_wheel.dae" scale="1 1 1"/>
+			</geometry>
+		</visual>
+	</link>
+	<joint name="rear_wheel_joint" type="continuous">
+		<origin xyz="-0.05 0 0.022" rpy="${pi/2} 0 0"/>
+		<axis xyz="0 0 1"/>
+		<parent link="chassic"/>
+		<child link="rear_wheel"/>
+	</joint>
 </robot>

Commit message: finalize import_obike.py extension & add color to meshes

File: data/urdf/robots/obike/urdf/obike.urdf (robot description, URDF)
Before this commit: robot obike, 9 links, 8 joints
Links:
- link chassic: mass None -> 0.288; geometry collision mesh filename=/home/teera/urdf/robots/obike/meshes/chassic.dae scale=1 1 1; visual mesh filename=/home/teera/urdf/robots/obike/meshes/chassic.dae scale=1 1 1
- link faulhaber: mass None -> 0.213; geometry visual mesh filename=/home/teera/urdf/robots/obike/meshes/faulhaber.dae scale=1 1 1
- link front_chassic: mass None -> 0.0298; geometry visual mesh filename=/home/teera/urdf/robots/obike/meshes/front_chassic.dae scale=1 1 1
- link front_wheel: mass None -> 0.0116; geometry collision mesh filename=/home/teera/urdf/robots/obike/meshes/front_wheel.dae scale=1 1 1; visual mesh filename=/home/teera/urdf/robots/obike/meshes/front_wheel.dae scale=1 1 1
- link front_wheel_arm: mass None -> 0.0043; geometry visual mesh filename=/home/teera/urdf/robots/obike/meshes/front_wheel_arm.dae scale=1 1 1
- link motor_mount: mass None -> 0.067; geometry visual mesh filename=/home/teera/urdf/robots/obike/meshes/motor_mount.dae scale=1 1 1
- link reaction_wheel: geometry visual mesh filename=/home/teera/urdf/robots/obike/meshes/reaction_wheel.dae scale=1 1 1
- link reaction_wheel_steel: mass None -> 0.198; geometry collision cylinder length=0.012 radius=0.0325; visual mesh filename=/home/teera/urdf/robots/obike/meshes/reaction_wheel_steel.d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 scale=1 1 1
- link rear_wheel: mass None -> 0.0273; geometry collision mesh filename=/home/teera/urdf/robots/obike/meshes/rear_wheel.dae scale=1 1 1; visual mesh filename=/home/teera/urdf/robots/obike/meshes/rear_wheel.dae scale=1 1 1

File: data/urdf/robots/obike/urdf/obike.xacro (robot description, xacro)
@@ -1,5 +1,5 @@
 <?xml version="1.0"?>
 <robot name="obike" xmlns:xacro="http://ros.org/wiki/xacro">
-	<xacro:property name="MODEL_PATH" value="/home/fiborobotlab/urdf/robots/obike/meshes/"/>
+	<xacro:property name="MODEL_PATH" value="/home/teera/urdf/robots/obike/meshes/"/>
     <xacro:macro name="inertial_box" params="size rho:=1000 xyz:='0 0 0' rpy:='0 0 0'">
 		<xacro:property name="w" value="${size.split()[0]}"/>
@@ -61,9 +61,9 @@
 		</collision>
 	</xacro:macro>
-	<xacro:macro name="inertial_manual" params="mass xyz:='0 0 0' rpy:='0 0 0' ixx iyy izz ixy:='0' ixz:='0' iyz:='0'">
-		<inertial>
-			<origin xyz="${xyz}" rpy="${rpy}"/>
-			<mass value="${mass}"/>
-			<inertia ixx="${ixx}" iyy="${iyy}" izz="${izz}" ixy="${ixy}" ixz="${ixz}" iyz="${iyz}"/>
+	<xacro:macro name="inertial_manual" params="mass xyz:='0 0 0' rpy:='0 0 0' ixx iyy izz iyz ixz ixy">
+		<inertial>
+			<origin xyz="${xyz}" rpy="${rpy}"/>
+			<mass value="${mass}"/>
+			<inertia ixx="${ixx}" iyy="${iyy}" izz="${izz}" iyz="${iyz}" ixz="${ixz}" ixy="${ixy}"/>
 		</inertial>
 	</xacro:macro>
@@ -74,4 +74,10 @@
 			</geometry>
 		</visual>
+		<xacro:inertial_manual mass="0.288" xyz="0.0047367 -0.00165617 0.0191097" ixx="3.80011e-05" iyy="8.50835e-05" izz="9.50647e-05" iyz="-1.16837e-11" ixz="-6.35148e-06" ixy="-3.93988e-11"/>
+		<collision>
+			<geometry>
+				<mesh filename="${MODEL_PATH}chassic.dae" scale="1 1 1"/>
+			</geometry>
+		</collision>
 	</link>
 	<link name="motor_mount">
@@ -81,4 +87,5 @@
 			</geometry>
 		</visual>
+		<xacro:inertial_manual mass="0.067" xyz="0.00311605 -2.39414e-08 -0.0261504" ixx="3.80011e-05" iyy="8.50835e-05" izz="9.50647e-05" iyz="-1.16837e-11" ixz="-6.35148e-06" ixy="-3.93988e-11"/>
 	</link>
 	<joint name="motor_mount_joint" type="fixed">
@@ -93,4 +100,10 @@
 			</geometry>
 		</visual>
+		<xacro:inertial_manual mass="0.0298" xyz="0.0277492 1.38661e-08 0.00859761" ixx="7.21055e-06" iyy="8.02622e-06" izz="1.19714e-05" iyz="-4.42397e-13" ixz="-1.61329e-06" ixy="5.32121e-12"/>
+		<!-- <collision>
+			<geometry>
+				<mesh filename="${MODEL_PATH}front_chassic.dae" scale="1 1 1"/>
+			</geometry>
+		</collision> -->
 	</link>
 	<joint name="front_chassic_joint" type="fixed">
@@ -105,4 +118,5 @@
 			</geometry>
 		</visual>
+		<xacro:inertial_manual mass="0.0043" xyz="-6.32629e-08 0.00613173 0.0206668" ixx="8.4523e-07" iyy="7.98604e-07" izz="1.47325e-07" iyz="-9.6622e-08" ixz="3.80111e-12" ixy="-2.0208e-12"/>
 	</link>
 	<joint name="front_wheel_arm_joint" type="continuous">
@@ -118,4 +132,10 @@
 			</geometry>
 		</visual>
+		<xacro:inertial_manual mass="0.0116" xyz="-9.22528e-13 -2.05375e-07 -0.000101895" ixx="1.52351e-06" iyy="1.52351e-06" izz="2.95246e-06" iyz="2.01001e-13" ixz="1.55876e-17" ixy="1.10854e-16"/>
+		<collision>
+			<geometry>
+				<mesh filename="${MODEL_PATH}front_wheel.dae" scale="1 1 1"/>
+			</geometry>
+		</collision>
 	</link>
 	<joint name="front_wheel_joint" type="continuous">
@@ -131,4 +151,5 @@
 			</geometry>
 		</visual>
+		<xacro:inertial_manual mass="0.213" xyz="4.82201e-09 -1.77912e-19 -0.0074239" ixx="0.000114919" iyy="0.000114919" izz="1.81057e-05" iyz="-9.40735e-22" ixz="1.44574e-11" ixy="3.73504e-22"/>
 	</link>
 	<joint name="faulhaber_joint" type="fixed">
@@ -143,4 +164,5 @@
 			</geometry>
 		</visual>
+		<!-- <xacro:inertial_manual mass="" xyz="" ixx="" iyy="" izz="" iyz="" ixz="" ixy=""/> -->
 	</link>
 	<joint name="reaction_wheel_joint" type="continuous">
@@ -156,4 +178,6 @@
 			</geometry>
 		</visual>
+		<xacro:inertial_manual mass="0.198" xyz="2.36685e-08 1.97235e-06 0.00337371" ixx="4.07098e-06" iyy="4.07082e-06" izz="7.53616e-06" iyz="1.64823e-10" ixz="1.77889e-12" ixy="-5.26622e-13"/>
+		<xacro:collision_cylinder length="0.012" radius="0.0325"/>
 	</link>
 	<joint name="reaction_wheel_steel_joint" type="fixed">
@@ -168,4 +192,10 @@
 			</geometry>
 		</visual>
+		<xacro:inertial_manual mass="0.0273" xyz="8.66222e-10 -2.46799e-07 -5.02853e-06" ixx="7.92469e-06" iyy="7.92468e-06" izz="1.53136e-05" iyz="1.27201e-13" ixz="-1.10104e-16" ixy="-1.1825e-17"/>
+		<collision>
+			<geometry>
+				<mesh filename="${MODEL_PATH}rear_wheel.dae" scale="1 1 1"/>
+			</geometry>
+		</collision>
 	</link>
 	<joint name="rear_wheel_joint" type="continuous">

Commit message: obike_lstm training (not finished)

File: data/urdf/robots/obike/urdf/obike.urdf (robot description, URDF)
Before this commit: robot obike, 9 links, 8 joints
Links:
- link chassic: geometry collision mesh filename=package://meshes/chassic.dae scale=1 1 1; visual mesh filename=package://meshes/chassic.dae scale=1 1 1
- link faulhaber: geometry visual mesh filename=package://meshes/faulhaber.dae scale=1 1 1
- link front_chassic: geometry visual mesh filename=package://meshes/front_chassic.dae scale=1 1 1
- link front_wheel: geometry collision mesh filename=package://meshes/front_wheel.dae scale=1 1 1; visual mesh filename=package://meshes/front_wheel.dae scale=1 1 1
- link front_wheel_arm: geometry visual mesh filename=package://meshes/front_wheel_arm.dae scale=1 1 1
- link motor_mount: geometry visual mesh filename=package://meshes/motor_mount.dae scale=1 1 1
- link reaction_wheel: geometry visual mesh filename=package://meshes/reaction_wheel.dae scale=1 1 1
- link reaction_wheel_steel: geometry collision cylinder length=0.012 radius=0.0325; visual mesh filename=package://meshes/reaction_wheel_steel.dae scale=1 1 1
- link rear_wheel: geometry collision mesh filename=package://meshes/rear_wheel.dae scale=1 1 1; visual mesh filename=package://meshes/rear_wheel.dae scale=1 1 1

File: data/urdf/robots/obike/urdf/obike.xacro (robot description, xacro)
@@ -1,5 +1,4 @@
 <?xml version="1.0"?>
 <robot name="obike" xmlns:xacro="http://ros.org/wiki/xacro">
-	<xacro:property name="MODEL_PATH" value="/home/teera/urdf/robots/obike/meshes/"/>
     <xacro:macro name="inertial_box" params="size rho:=1000 xyz:='0 0 0' rpy:='0 0 0'">
 		<xacro:property name="w" value="${size.split()[0]}"/>
@@ -71,5 +70,5 @@
 		<visual>
 			<geometry>
-				<mesh filename="${MODEL_PATH}chassic.dae" scale="1 1 1"/>
+				<mesh filename="package://meshes/chassic.dae" scale="1 1 1"/>
 			</geometry>
 		</visual>
@@ -77,5 +76,5 @@
 		<collision>
 			<geometry>
-				<mesh filename="${MODEL_PATH}chassic.dae" scale="1 1 1"/>
+				<mesh filename="package://meshes/chassic.dae" scale="1 1 1"/>
 			</geometry>
 		</collision>
@@ -84,5 +83,5 @@
 		<visual>
 			<geometry>
-				<mesh filename="${MODEL_PATH}motor_mount.dae" scale="1 1 1"/>
+				<mesh filename="package://meshes/motor_mount.dae" scale="1 1 1"/>
 			</geometry>
 		</visual>
@@ -97,5 +96,5 @@
 		<visual>
 			<geometry>
-				<mesh filename="${MODEL_PATH}front_chassic.dae" scale="1 1 1"/>
+				<mesh filename="package://meshes/front_chassic.dae" scale="1 1 1"/>
 			</geometry>
 		</visual>
@@ -103,5 +102,5 @@
 		<!-- <collision>
 			<geometry>
-				<mesh filename="${MODEL_PATH}front_chassic.dae" scale="1 1 1"/>
+				<mesh filename="package://meshes/front_chassic.dae" scale="1 1 1"/>
 			</geometry>
 		</collision> -->
@@ -115,5 +114,5 @@
 		<visual>
 			<geometry>
-				<mesh filename="${MODEL_PATH}front_wheel_arm.dae" scale="1 1 1"/>
+				<mesh filename="package://meshes/front_wheel_arm.dae" scale="1 1 1"/>
 			</geometry>
 		</visual>
@@ -129,5 +128,5 @@
 		<visual>
 			<geometry>
-				<mesh filename="${MODEL_PATH}front_wheel.dae" scale="1 1 1"/>
+				<mesh filename="package://meshes/front_wheel.dae" scale="1 1 1"/>
 			</geometry>
 		</visual>
@@ -135,5 +134,5 @@
 		<collision>
 			<geometry>
-				<mesh filename="${MODEL_PATH}front_wheel.dae" scale="1 1 1"/>
+				<mesh filename="package://meshes/front_wheel.dae" scale="1 1 1"/>
 			</geometry>
 		</collision>
@@ -148,5 +147,5 @@
 		<visual>
 			<geometry>
-				<mesh filename="${MODEL_PATH}faulhaber.dae" scale="1 1 1"/>
+				<mesh filename="package://meshes/faulhaber.dae" scale="1 1 1"/>
 			</geometry>
 		</visual>
@@ -161,5 +160,5 @@
 		<visual>
 			<geometry>
-				<mesh filename="${MODEL_PATH}reaction_wheel.dae" scale="1 1 1"/>
+				<mesh filename="package://meshes/reaction_wheel.dae" scale="1 1 1"/>
 			</geometry>
 		</visual>
@@ -175,5 +174,5 @@
 		<visual>
 			<geometry>
-				<mesh filename="${MODEL_PATH}reaction_wheel_steel.dae" scale="1 1 1"/>
+				<mesh filename="package://meshes/reaction_wheel_steel.dae" scale="1 1 1"/>
 			</geometry>
 		</visual>
@@ -189,5 +188,5 @@
 		<visual>
 			<geometry>
-				<mesh filename="${MODEL_PATH}rear_wheel.dae" scale="1 1 1"/>
+				<mesh filename="package://meshes/rear_wheel.dae" scale="1 1 1"/>
 			</geometry>
 		</visual>
@@ -195,5 +194,5 @@
 		<collision>
 			<geometry>
-				<mesh filename="${MODEL_PATH}rear_wheel.dae" scale="1 1 1"/>
+				<mesh filename="package://meshes/rear_wheel.dae" scale="1 1 1"/>
 			</geometry>
 		</collision>
